File: Hardware/RCCAR_IF_Board_GPS/RCCAR_IF_Board_GPS.kicad_pcb (KiCad board)
At the start: 4 copper layers, 81 x 55 mm, 169 parts, among them J1 SMA, J2 SMA, J3 SMA, P1 POWER, P11 OUT_1, P12 OUT_2, P13 USB_UBLOX, P14 OUT_3, P15 OUT_4, P2 USB_STM, P3 I2C, P4 UART, P5 NRF_SPI, P6 SWD, P7 ADC_GPIO, P8 CAN, P9 CAN, SW1 Address, U1 STM32F40X_LQFP100, U10 I2C_VOLTAGE, U11 USB_SUPPLY, U12 AP131-33, U13 ublox_neo_m8p, U2 CC2520, U3 CC2592, U4 CC1120, U5 MCP16311/2, U6 MCP16311/2, U7 TJA1051TK3, U8 MPU9150, U9 USB_SUPPLY, X1 8M, X2 32M, X3 32M

Commit message: Updated PCB with MPU9250
Parts:
- added C76: 100n, Capacitors_SMD:C_0603, F.Cu at (118.5, 95.4)
- added C77: 2.2u, Capacitors_SMD:C_0603, F.Cu at (120.9, 99.3)
- added C78: 2.2u, Capacitors_SMD:C_0603, F.Cu at (115.6, 98.3)
- added U14: MPU9250, Housings_DFN_QFN:QFN-24_3x3mm_Pitch0.4mm, F.Cu at (118.4, 98.2)
- R20: value 10R -> 4.7R
- moved C65 3.28 mm to (122.6, 102.0), turned to 315 degrees
- moved R26 3.18 mm to (121.5, 96.9)
- moved R27 3.05 mm to (123.1, 97.7)
Connections:
- P13 pad 4: (no net) -> Net-(P13-Pad4)
- P2 pad 4: (no net) -> Net-(P2-Pad4)
- P6 pad 1: (no net) -> Net-(P6-Pad1)
- U1 pad 1: (no net) -> Net-(U1-Pad1)
- U1 pad 2: (no net) -> Net-(U1-Pad2)
- U1 pad 3: (no net) -> Net-(U1-Pad3)
- U1 pad 33: (no net) -> Net-(U1-Pad33)
- U1 pad 34: (no net) -> Net-(U1-Pad34)
- U1 pad 37: (no net) -> Net-(U1-Pad37)
- U1 pad 38: (no net) -> Net-(U1-Pad38)
- U1 pad 55: (no net) -> Net-(U1-Pad55)
- U1 pad 61: (no net) -> Net-(U1-Pad61)
- U1 pad 67: (no net) -> Net-(U1-Pad67)
- U1 pad 69: (no net) -> Net-(U1-Pad69)
- U1 pad 7: (no net) -> Net-(U1-Pad7)
- U1 pad 77: (no net) -> Net-(U1-Pad77)
- U1 pad 8: (no net) -> Net-(U1-Pad8)
- U1 pad 86: (no net) -> Net-(U1-Pad86)
- U1 pad 87: (no net) -> Net-(U1-Pad87)
- U1 pad 88: (no net) -> Net-(U1-Pad88)
- U1 pad 89: (no net) -> Net-(U1-Pad89)
- U1 pad 9: (no net) -> Net-(U1-Pad9)
- U1 pad 90: (no net) -> Net-(U1-Pad90)
- U1 pad 91: (no net) -> Net-(U1-Pad91)
- U11 pad 3: (no net) -> Net-(U11-Pad3)
- U12 pad 4: (no net) -> Net-(U12-Pad4)
- U13 pad 1: (no net) -> Net-(U13-Pad1)
- U13 pad 14: (no net) -> Net-(U13-Pad14)
- U13 pad 16: (no net) -> Net-(U13-Pad16)
- U13 pad 17: (no net) -> Net-(U13-Pad17)
- U13 pad 18: (no net) -> Net-(U13-Pad18)
- U13 pad 19: (no net) -> Net-(U13-Pad19)
- U13 pad 2: (no net) -> Net-(U13-Pad2)
- U13 pad 4: (no net) -> Net-(U13-Pad4)
- U2 pad 18: (no net) -> Net-(U2-Pad18)
- U4 pad 16: (no net) -> Net-(U4-Pad16)
- U8 pad 1: (no net) -> Net-(U8-Pad1)
- U8 pad 11: (no net) -> Net-(U8-Pad11)
- U8 pad 12: (no net) -> Net-(U8-Pad12)
- U8 pad 22: (no net) -> Net-(U8-Pad22)
- U8 pad 6: (no net) -> Net-(U8-Pad6)
- U8 pad 7: (no net) -> Net-(U8-Pad7)
- U9 pad 3: (no net) -> Net-(U9-Pad3)
Routing:
- net GND: track 1201.0 -> 1215.2 mm, vias 303 -> 304
- net VCC: track 376.5 -> 386.0 mm
- net Net-(C65-Pad1): track 1.63 -> 3.95 mm
- net /MCU/PB11_SDA2: track 36.9 -> 38.9 mm, vias 2 -> 5
- net /MCU/PB10_SCL2: track 36.9 -> 38.6 mm, vias 2 -> 4
- net Net-(C76-Pad1): track 0.00 -> 1.47 mm
Other:
- net class Default: trace_width 0.20066 -> 0.25
- board text added: "RTK Controller V1.2"
- board text removed: "RTK Controller V1.1"
- board text removed: "SP Technical Research Institute of Sweden"
