File: Hardware/RCCAR_IF_Board_GPS/CAN.sch (KiCad schematic (older format))
At the start: 4 parts, among them U7 TJA1051TK3

Commit message: Added gitignore files
Parts:
- C63, C73: symbol C -> RCCAR_IF_Board_GPS-rescue:C-RESCUE-RCCAR_IF_Board_GPS
- R19: symbol R -> RCCAR_IF_Board_GPS-rescue:R-RESCUE-RCCAR_IF_Board_GPS
- U7: symbol TJA1051TK3 -> crf_1:TJA1051TK3
Changed lines of the file:
@@
-EESchema Schematic File Version 2
-LIBS:RCCAR_IF_Board_GPS-rescue
-LIBS:power
-LIBS:device
-LIBS:transistors
-LIBS:conn
-LIBS:linear
-LIBS:regul
-LIBS:74xx
-LIBS:cmos4000
-LIBS:adc-dac
-LIBS:memory
-LIBS:xilinx
-LIBS:microcontrollers
-LIBS:dsp
-LIBS:microchip
-LIBS:analog_switches
-LIBS:motorola
-LIBS:texas
-LIBS:intel
-LIBS:audio
-LIBS:interface
-LIBS:digital-audio
-LIBS:philips
-LIBS:display
-LIBS:cypress
-LIBS:siliconi
-LIBS:opto
-LIBS:atmel
-LIBS:contrib
-LIBS:valves
-LIBS:crf_1
-LIBS:dips-s
+EESchema Schematic File Version 4
 LIBS:RCCAR_IF_Board_GPS-cache
 EELAYER 26 0
@@
 $EndDescr
 $Comp
-L VCC #PWR099
+L power:VCC #PWR099
 U 1 1 56C0C064
 P 6600 3600
@@
 Connection ~ 7150 3750
 $Comp
-L C C63
+L RCCAR_IF_Board_GPS-rescue:C-RESCUE-RCCAR_IF_Board_GPS C63
 U 1 1 56C0C165
 P 6600 4450
@@
 $EndComp
 $Comp
-L R R19
+L RCCAR_IF_Board_GPS-rescue:R-RESCUE-RCCAR_IF_Board_GPS R19
 U 1 1 56C0C2A3
 P 7150 4000
@@
 	7150 4150 7150 4250
 $Comp
-L GND #PWR0100
+L power:GND #PWR0100
 U 1 1 56C0C32A
 P 5900 4800
@@
 	5900 4450 5900 4800
 $Comp
-L TJA1051TK3 U7
+L crf_1:TJA1051TK3 U7
 U 1 1 585B3B77
 P 5900 4000
@@
 Connection ~ 5900 4700
 $Comp
-L C C73
+L RCCAR_IF_Board_GPS-rescue:C-RESCUE-RCCAR_IF_Board_GPS C73
 U 1 1 585B3FED
 P 4750 4450
@@
 Connection ~ 6450 4700
 $Comp
-L +5V #PWR0101
+L power:+5V #PWR0101
 U 1 1 585B425F
 P 4750 3600
