File: Hardware/RCCAR_IF_Board_GPS/CC1120.sch (KiCad schematic (older format))
At the start: 39 parts, among them J2 SMA, U4 CC1120, X3 32M

Commit message: Added gitignore files
Parts:
- C27, C28, C29, C30, C31, C32, C33, C34, C35, C36, C37, C38, C39, C40, C41, C42, C43, C44, C45, C46, C47, C48, C49, C50, C51: symbol C -> RCCAR_IF_Board_GPS-rescue:C-RESCUE-RCCAR_IF_Board_GPS
- J2: symbol SMA -> crf_1:SMA
- L10, L11, L12, L13, L5, L6, L7, L8, L9: symbol INDUCTOR_SMALL -> crf_1:INDUCTOR_SMALL
- R11, R12: symbol R -> RCCAR_IF_Board_GPS-rescue:R-RESCUE-RCCAR_IF_Board_GPS
- U4: symbol CC1120 -> crf_1:CC1120
- X3: symbol Crystal_GND3 -> RCCAR_IF_Board_GPS-rescue:Crystal_GND3-RESCUE-RCCAR_IF_Board_GPS
Changed lines of the file:
@@
-EESchema Schematic File Version 2
-LIBS:RCCAR_IF_Board_GPS-rescue
-LIBS:power
-LIBS:device
-LIBS:transistors
-LIBS:conn
-LIBS:linear
-LIBS:regul
-LIBS:74xx
-LIBS:cmos4000
-LIBS:adc-dac
-LIBS:memory
-LIBS:xilinx
-LIBS:microcontrollers
-LIBS:dsp
-LIBS:microchip
-LIBS:analog_switches
-LIBS:motorola
-LIBS:texas
-LIBS:intel
-LIBS:audio
-LIBS:interface
-LIBS:digital-audio
-LIBS:philips
-LIBS:display
-LIBS:cypress
-LIBS:siliconi
-LIBS:opto
-LIBS:atmel
-LIBS:contrib
-LIBS:valves
-LIBS:crf_1
-LIBS:dips-s
+EESchema Schematic File Version 4
 LIBS:RCCAR_IF_Board_GPS-cache
 EELAYER 26 0
@@
 $EndDescr
 $Comp
-L CC1120 U4
+L crf_1:CC1120 U4
 U 1 1 56BC1F3C
 P 3250 3550
@@
 $EndComp
 $Comp
-L GND #PWR078
+L power:GND #PWR078
 U 1 1 56BC9D42
 P 2550 1850
@@
 $EndComp
 $Comp
-L C C30
+L RCCAR_IF_Board_GPS-rescue:C-RESCUE-RCCAR_IF_Board_GPS C30
 U 1 1 56BC9D9E
 P 1900 1350
@@
 $EndComp
 $Comp
-L C C31
+L RCCAR_IF_Board_GPS-rescue:C-RESCUE-RCCAR_IF_Board_GPS C31
 U 1 1 56BC9DCA
 P 1900 2150
@@
 $EndComp
 $Comp
-L GND #PWR079
+L power:GND #PWR079
 U 1 1 56BC9E4D
 P 1650 2400
@@
 $EndComp
 $Comp
-L GND #PWR080
+L power:GND #PWR080
 U 1 1 56BC9F09
 P 2150 2400
@@
 $EndComp
 $Comp
-L C C32
+L RCCAR_IF_Board_GPS-rescue:C-RESCUE-RCCAR_IF_Board_GPS C32
 U 1 1 56BC9FCB
 P 3200 1150
@@
 $EndComp
 $Comp
-L C C34
+L RCCAR_IF_Board_GPS-rescue:C-RESCUE-RCCAR_IF_Board_GPS C34
 U 1 1 56BCA488
 P 3500 1150
@@
 $EndComp
 $Comp
-L GND #PWR081
+L power:GND #PWR081
 U 1 1 56BCA4F1
 P 3850 1200
@@
 $EndComp
 $Comp
-L C C36
+L RCCAR_IF_Board_GPS-rescue:C-RESCUE-RCCAR_IF_Board_GPS C36
 U 1 1 56BCA605
 P 3950 1950
@@
 $EndComp
 $Comp
-L C C38
+L RCCAR_IF_Board_GPS-rescue:C-RESCUE-RCCAR_IF_Board_GPS C38
 U 1 1 56BCA652
 P 4250 1950
@@
 $EndComp
 $Comp
-L C C39
+L RCCAR_IF_Board_GPS-rescue:C-RESCUE-RCCAR_IF_Board_GPS C39
 U 1 1 56BCA682
 P 4550 1950
@@
 $EndComp
 $Comp
-L GND #PWR082
+L power:GND #PWR082
 U 1 1 56BCA798
 P 4550 2300
@@
 $EndComp
 $Comp
-L C C27
+L RCCAR_IF_Board_GPS-rescue:C-RESCUE-RCCAR_IF_Board_GPS C27
 U 1 1 56BCAE40
 P 1350 3200
@@
 $EndComp
 $Comp
-L C C28
+L RCCAR_IF_Board_GPS-rescue:C-RESCUE-RCCAR_IF_Board_GPS C28
 U 1 1 56BCAF48
 P 1350 3600
@@
 $EndComp
 $Comp
-L GND #PWR083
+L power:GND #PWR083
 U 1 1 56BCB1BE
 P 950 3750
@@
 $EndComp
 $Comp
-L C C29
+L RCCAR_IF_Board_GPS-rescue:C-RESCUE-RCCAR_IF_Board_GPS C29
 U 1 1 56BCB675
 P 1600 4000
@@
 $EndComp
 $Comp
-L GND #PWR084
+L power:GND #PWR084
 U 1 1 56BCB7EA
 P 1600 4300
@@
 $EndComp
 $Comp
-L C C33
+L RCCAR_IF_Board_GPS-rescue:C-RESCUE-RCCAR_IF_Board_GPS C33
 U 1 1 56BCC315
 P 3200 5200
@@
 $EndComp
 $Comp
-L C C35
+L RCCAR_IF_Board_GPS-rescue:C-RESCUE-RCCAR_IF_Board_GPS C35
 U 1 1 56BCC3CE
 P 3500 5200
@@
 $EndComp
 $Comp
-L R R11
+L RCCAR_IF_Board_GPS-rescue:R-RESCUE-RCCAR_IF_Board_GPS R11
 U 1 1 56BCC4AE
 P 3800 5200
@@
 $EndComp
 $Comp
-L C C37
+L RCCAR_IF_Board_GPS-rescue:C-RESCUE-RCCAR_IF_Board_GPS C37
 U 1 1 56BCC89B
 P 4100 5200
@@
 $EndComp
 $Comp
-L GND #PWR085
+L power:GND #PWR085
 U 1 1 56BCCF22
 P 3200 5600
@@
 CS_N
 $Comp
-L C C40
+L RCCAR_IF_Board_GPS-rescue:C-RESCUE-RCCAR_IF_Board_GPS C40
 U 1 1 56BCE68D
 P 4700 3050
@@
 $EndComp
 $Comp
-L C C41
+L RCCAR_IF_Board_GPS-rescue:C-RESCUE-RCCAR_IF_Board_GPS C41
 U 1 1 56BCE8DE
 P 5150 3050
@@
 	5150 2700 5150 2900
 $Comp
-L GND #PWR086
+L power:GND #PWR086
 U 1 1 56BCEAE8
 P 5150 3250
@@
 	5150 3200 5150 3250
 $Comp
-L C C43
+L RCCAR_IF_Board_GPS-rescue:C-RESCUE-RCCAR_IF_Board_GPS C43
 U 1 1 56BCF209
 P 5550 3050
@@
 Connection ~ 5150 2800
 $Comp
-L GND #PWR087
+L power:GND #PWR087
 U 1 1 56BCF6F6
 P 5550 3250
@@
 	5550 3200 5550 3250
 $Comp
-L INDUCTOR_SMALL L6
+L crf_1:INDUCTOR_SMALL L6
 U 1 1 56BCFC13
 P 6150 3450
@@
 $EndComp
 $Comp
-L INDUCTOR_SMALL L9
+L crf_1:INDUCTOR_SMALL L9
 U 1 1 56BD02E6
 P 7100 3050
@@
 $EndComp
 $Comp
-L INDUCTOR_SMALL L10
+L crf_1:INDUCTOR_SMALL L10
 U 1 1 56BD03FB
 P 7100 4050
@@
 $EndComp
 $Comp
-L C C49
+L RCCAR_IF_Board_GPS-rescue:C-RESCUE-RCCAR_IF_Board_GPS C49
 U 1 1 56BD0471
 P 7100 2650
@@
 Connection ~ 6600 3050
 $Comp
-L GND #PWR088
+L power:GND #PWR088
 U 1 1 56BD0935
 P 7500 2800
@@
 	7500 2650 7500 2800
 $Comp
-L C C48
+L RCCAR_IF_Board_GPS-rescue:C-RESCUE-RCCAR_IF_Board_GPS C48
 U 1 1 56BD0A0A
 P 7000 3800
@@
 	7800 3800 7150 3800
 $Comp
-L GND #PWR089
+L power:GND #PWR089
 U 1 1 56BD0C86
 P 7500 4150
@@
 	7500 4050 7500 4150
 $Comp
-L INDUCTOR_SMALL L12
+L crf_1:INDUCTOR_SMALL L12
 U 1 1 56BD0D85
 P 8050 3850
@@
 	8050 4450 8050 4100
 $Comp
-L C C50
+L RCCAR_IF_Board_GPS-rescue:C-RESCUE-RCCAR_IF_Board_GPS C50
 U 1 1 56BD11F2
 P 7300 4750
@@
 Connection ~ 7300 4450
 $Comp
-L INDUCTOR_SMALL L7
+L crf_1:INDUCTOR_SMALL L7
 U 1 1 56BD147C
 P 6450 5000
@@
 $EndComp
 $Comp
-L INDUCTOR_SMALL L11
+L crf_1:INDUCTOR_SMALL L11
 U 1 1 56BD1C41
 P 7950 5000
@@
 Connection ~ 7300 5000
 $Comp
-L C C47
+L RCCAR_IF_Board_GPS-rescue:C-RESCUE-RCCAR_IF_Board_GPS C47
 U 1 1 56BD1F48
 P 6450 5300
@@
 Connection ~ 6850 5000
 $Comp
-L C C44
+L RCCAR_IF_Board_GPS-rescue:C-RESCUE-RCCAR_IF_Board_GPS C44
 U 1 1 56BD2662
 P 5700 5000
@@
 	5250 5000 5550 5000
 $Comp
-L INDUCTOR_SMALL L5
+L crf_1:INDUCTOR_SMALL L5
 U 1 1 56BD2DF8
 P 5250 5450
@@
 Connection ~ 5250 5000
 $Comp
-L INDUCTOR_SMALL L13
+L crf_1:INDUCTOR_SMALL L13
 U 1 1 56BD38DF
 P 9100 5000
@@
 	8200 5000 8850 5000
 $Comp
-L C C51
+L RCCAR_IF_Board_GPS-rescue:C-RESCUE-RCCAR_IF_Board_GPS C51
 U 1 1 56BD3D0C
 P 8500 5350
@@
 $EndComp
 $Comp
-L GND #PWR090
+L power:GND #PWR090
 U 1 1 56BD3EB1
 P 8500 5600
@@
 Connection ~ 8500 5000
 $Comp
-L SMA J2
+L crf_1:SMA J2
 U 1 1 56BD40EA
 P 9750 5100
@@
 	9350 5000 9650 5000
 $Comp
-L GND #PWR091
+L power:GND #PWR091
 U 1 1 56BD4289
 P 9850 5400
@@
 Connection ~ 9750 5300
 $Comp
-L R R12
+L RCCAR_IF_Board_GPS-rescue:R-RESCUE-RCCAR_IF_Board_GPS R12
 U 1 1 56BD5583
 P 5500 6050
@@
 $EndComp
 $Comp
-L C C45
+L RCCAR_IF_Board_GPS-rescue:C-RESCUE-RCCAR_IF_Board_GPS C45
 U 1 1 56BD56DA
 P 5800 6050
@@
 Connection ~ 5500 6350
 $Comp
-L C C42
+L RCCAR_IF_Board_GPS-rescue:C-RESCUE-RCCAR_IF_Board_GPS C42
 U 1 1 56BD5EAE
 P 5500 6650
@@
 $EndComp
 $Comp
-L C C46
+L RCCAR_IF_Board_GPS-rescue:C-RESCUE-RCCAR_IF_Board_GPS C46
 U 1 1 56BD5F96
 P 5800 6650
@@
 Connection ~ 5800 6350
 $Comp
-L GND #PWR092
+L power:GND #PWR092
 U 1 1 56BD62D8
 P 5800 6950
@@
 Connection ~ 5800 6850
 $Comp
-L VCC #PWR093
+L power:VCC #PWR093
 U 1 1 56BD84C6
 P 6650 1600
@@
 $EndComp
 $Comp
-L INDUCTOR_SMALL L8
+L crf_1:INDUCTOR_SMALL L8
 U 1 1 56BD8543
 P 7050 1750
@@
 	7300 1750 7950 1750
 $Comp
-L PWR_FLAG #FLG094
+L power:PWR_FLAG #FLG094
 U 1 1 56C814C1
 P 7600 1600
@@
 Connection ~ 7600 1750
 $Comp
-L Crystal_GND3 X3
+L RCCAR_IF_Board_GPS-rescue:Crystal_GND3-RESCUE-RCCAR_IF_Board_GPS X3
 U 1 1 585F52F5
 P 2150 1750
