File: Hardware/RCCAR_IF_Board_GPS/CC2520.sch (KiCad schematic (older format))
At the start: 29 parts, among them J1 SMA, U2 CC2520, U3 CC2592, X2 32M

Commit message: Added gitignore files
Parts:
- C13, C14, C15, C16, C17, C18, C19, C20, C21, C22, C23, C24, C25, C26, C70, C71, C72: symbol C -> RCCAR_IF_Board_GPS-rescue:C-RESCUE-RCCAR_IF_Board_GPS
- J1: symbol SMA -> crf_1:SMA
- L15, L17, L2, L3, L4: symbol INDUCTOR_SMALL -> crf_1:INDUCTOR_SMALL
- R4, R5, R8: symbol R -> RCCAR_IF_Board_GPS-rescue:R-RESCUE-RCCAR_IF_Board_GPS
- U2: symbol CC2520 -> crf_1:CC2520
- U3: symbol CC2592 -> crf_1:CC2592
- X2: symbol Crystal_GND3 -> RCCAR_IF_Board_GPS-rescue:Crystal_GND3-RESCUE-RCCAR_IF_Board_GPS
Changed lines of the file:
@@
-EESchema Schematic File Version 2
-LIBS:RCCAR_IF_Board_GPS-rescue
-LIBS:power
-LIBS:device
-LIBS:transistors
-LIBS:conn
-LIBS:linear
-LIBS:regul
-LIBS:74xx
-LIBS:cmos4000
-LIBS:adc-dac
-LIBS:memory
-LIBS:xilinx
-LIBS:microcontrollers
-LIBS:dsp
-LIBS:microchip
-LIBS:analog_switches
-LIBS:motorola
-LIBS:texas
-LIBS:intel
-LIBS:audio
-LIBS:interface
-LIBS:digital-audio
-LIBS:philips
-LIBS:display
-LIBS:cypress
-LIBS:siliconi
-LIBS:opto
-LIBS:atmel
-LIBS:contrib
-LIBS:valves
-LIBS:crf_1
-LIBS:dips-s
+EESchema Schematic File Version 4
 LIBS:RCCAR_IF_Board_GPS-cache
 EELAYER 26 0
@@
 $EndDescr
 $Comp
-L CC2520 U2
+L crf_1:CC2520 U2
 U 1 1 56BB4EB8
 P 2700 3850
@@
 $EndComp
 $Comp
-L VCC #PWR052
+L power:VCC #PWR052
 U 1 1 56BB4ECB
 P 5600 1450
@@
 CC_RESET
 $Comp
-L C C16
+L RCCAR_IF_Board_GPS-rescue:C-RESCUE-RCCAR_IF_Board_GPS C16
 U 1 1 56BB56FC
 P 4550 5400
@@
 $EndComp
 $Comp
-L C C18
+L RCCAR_IF_Board_GPS-rescue:C-RESCUE-RCCAR_IF_Board_GPS C18
 U 1 1 56BB5754
 P 5200 5400
@@
 $EndComp
 $Comp
-L R R5
+L RCCAR_IF_Board_GPS-rescue:R-RESCUE-RCCAR_IF_Board_GPS R5
 U 1 1 56BB5842
 P 3850 5350
@@
 $EndComp
 $Comp
-L GND #PWR053
+L power:GND #PWR053
 U 1 1 56BB593C
 P 1600 5400
@@
 $EndComp
 $Comp
-L GND #PWR054
+L power:GND #PWR054
 U 1 1 56BB596F
 P 3850 5600
@@
 $EndComp
 $Comp
-L GND #PWR055
+L power:GND #PWR055
 U 1 1 56BB599B
 P 4550 5600
@@
 $EndComp
 $Comp
-L GND #PWR056
+L power:GND #PWR056
 U 1 1 56BB59C7
 P 5200 5600
@@
 $EndComp
 $Comp
-L GND #PWR057
+L power:GND #PWR057
 U 1 1 56BB5D07
 P 4150 4450
@@
 $EndComp
 $Comp
-L C C13
+L RCCAR_IF_Board_GPS-rescue:C-RESCUE-RCCAR_IF_Board_GPS C13
 U 1 1 56BB5D30
 P 3900 4350
@@
 $EndComp
 $Comp
-L C C14
+L RCCAR_IF_Board_GPS-rescue:C-RESCUE-RCCAR_IF_Board_GPS C14
 U 1 1 56BB63A2
 P 4000 2100
@@
 $EndComp
 $Comp
-L C C15
+L RCCAR_IF_Board_GPS-rescue:C-RESCUE-RCCAR_IF_Board_GPS C15
 U 1 1 56BB64BB
 P 4550 2100
@@
 $EndComp
 $Comp
-L C C17
+L RCCAR_IF_Board_GPS-rescue:C-RESCUE-RCCAR_IF_Board_GPS C17
 U 1 1 56BB64F3
 P 5150 2100
@@
 $EndComp
 $Comp
-L C C19
+L RCCAR_IF_Board_GPS-rescue:C-RESCUE-RCCAR_IF_Board_GPS C19
 U 1 1 56BB652A
 P 5600 1850
@@
 $EndComp
 $Comp
-L R R4
+L RCCAR_IF_Board_GPS-rescue:R-RESCUE-RCCAR_IF_Board_GPS R4
 U 1 1 56BB6707
 P 1550 2600
@@
 $EndComp
 $Comp
-L GND #PWR058
+L power:GND #PWR058
 U 1 1 56BB6C68
 P 4000 2350
@@
 $EndComp
 $Comp
-L GND #PWR059
+L power:GND #PWR059
 U 1 1 56BB6CB5
 P 4550 2350
@@
 $EndComp
 $Comp
-L GND #PWR060
+L power:GND #PWR060
 U 1 1 56BB6CE1
 P 5150 2350
@@
 $EndComp
 $Comp
-L CC2592 U3
+L crf_1:CC2592 U3
 U 1 1 56BB7634
 P 6100 3700
@@
 $EndComp
 $Comp
-L R R8
+L RCCAR_IF_Board_GPS-rescue:R-RESCUE-RCCAR_IF_Board_GPS R8
 U 1 1 56BB7908
 P 6850 4300
@@
 $EndComp
 $Comp
-L GND #PWR061
+L power:GND #PWR061
 U 1 1 56BB79D8
 P 6850 4600
@@
 $EndComp
 $Comp
-L GND #PWR062
+L power:GND #PWR062
 U 1 1 56BB7A57
 P 5400 4600
@@
 Connection ~ 5400 4400
 $Comp
-L GND #PWR063
+L power:GND #PWR063
 U 1 1 56BB8384
 P 5600 2350
@@
 $EndComp
 $Comp
-L C C20
+L RCCAR_IF_Board_GPS-rescue:C-RESCUE-RCCAR_IF_Board_GPS C20
 U 1 1 56BB87A2
 P 7050 3050
@@
 $EndComp
 $Comp
-L C C21
+L RCCAR_IF_Board_GPS-rescue:C-RESCUE-RCCAR_IF_Board_GPS C21
 U 1 1 56BB8818
 P 7400 3050
@@
 $EndComp
 $Comp
-L C C22
+L RCCAR_IF_Board_GPS-rescue:C-RESCUE-RCCAR_IF_Board_GPS C22
 U 1 1 56BB885F
 P 7750 3050
@@
 Connection ~ 7050 2800
 $Comp
-L GND #PWR064
+L power:GND #PWR064
 U 1 1 56BB9357
 P 7050 3250
@@
 $EndComp
 $Comp
-L GND #PWR065
+L power:GND #PWR065
 U 1 1 56BB9392
 P 7400 3250
@@
 $EndComp
 $Comp
-L GND #PWR066
+L power:GND #PWR066
 U 1 1 56BB93CD
 P 7750 3250
@@
 	7750 3200 7750 3250
 $Comp
-L INDUCTOR_SMALL L2
+L crf_1:INDUCTOR_SMALL L2
 U 1 1 56BB9D8A
 P 8100 3150
@@
 $EndComp
 $Comp
-L INDUCTOR_SMALL L3
+L crf_1:INDUCTOR_SMALL L3
 U 1 1 56BBA330
 P 8600 3500
@@
 $EndComp
 $Comp
-L INDUCTOR_SMALL L4
+L crf_1:INDUCTOR_SMALL L4
 U 1 1 56BBA4CB
 P 9400 3500
@@
 	8850 3500 9150 3500
 $Comp
-L C C23
+L RCCAR_IF_Board_GPS-rescue:C-RESCUE-RCCAR_IF_Board_GPS C23
 U 1 1 56BBAE6D
 P 8100 3800
@@
 $EndComp
 $Comp
-L C C24
+L RCCAR_IF_Board_GPS-rescue:C-RESCUE-RCCAR_IF_Board_GPS C24
 U 1 1 56BBAF24
 P 9050 3800
@@
 $EndComp
 $Comp
-L C C26
+L RCCAR_IF_Board_GPS-rescue:C-RESCUE-RCCAR_IF_Board_GPS C26
 U 1 1 56BBAF95
 P 9950 3800
@@
 $EndComp
 $Comp
-L C C25
+L RCCAR_IF_Board_GPS-rescue:C-RESCUE-RCCAR_IF_Board_GPS C25
 U 1 1 56BBB03A
 P 9950 3150
@@
 $EndComp
 $Comp
-L SMA J1
+L crf_1:SMA J1
 U 1 1 56BBB2F7
 P 9850 2600
@@
 Connection ~ 9050 3500
 $Comp
-L GND #PWR067
+L power:GND #PWR067
 U 1 1 56BBB6F9
 P 8100 4100
@@
 $EndComp
 $Comp
-L GND #PWR068
+L power:GND #PWR068
 U 1 1 56BBB74C
 P 9050 4100
@@
 $EndComp
 $Comp
-L GND #PWR069
+L power:GND #PWR069
 U 1 1 56BBB79F
 P 9950 4100
@@
 	8100 4100 8100 3950
 $Comp
-L GND #PWR070
+L power:GND #PWR070
 U 1 1 56BBBA86
 P 9600 2750
@@
 	4550 5050 4700 5050
 $Comp
-L GND #PWR071
+L power:GND #PWR071
 U 1 1 56BC9850
 P 4850 5350
@@
 	4850 5250 4850 5350
 $Comp
-L INDUCTOR_SMALL L15
+L crf_1:INDUCTOR_SMALL L15
 U 1 1 56BCD877
 P 4400 3500
@@
 Do\nnot\nmount
 $Comp
-L INDUCTOR_SMALL L17
+L crf_1:INDUCTOR_SMALL L17
 U 1 1 56C289F8
 P 8150 5050
@@
 $EndComp
 $Comp
-L C C70
+L RCCAR_IF_Board_GPS-rescue:C-RESCUE-RCCAR_IF_Board_GPS C70
 U 1 1 56C28F61
 P 8650 5300
@@
 $EndComp
 $Comp
-L VCC #PWR072
+L power:VCC #PWR072
 U 1 1 56C293DC
 P 7700 4850
@@
 $EndComp
 $Comp
-L C C71
+L RCCAR_IF_Board_GPS-rescue:C-RESCUE-RCCAR_IF_Board_GPS C71
 U 1 1 56C29527
 P 9000 5300
@@
 $EndComp
 $Comp
-L C C72
+L RCCAR_IF_Board_GPS-rescue:C-RESCUE-RCCAR_IF_Board_GPS C72
 U 1 1 56C295FD
 P 9350 5300
@@
 Connection ~ 8650 5050
 $Comp
-L GND #PWR073
+L power:GND #PWR073
 U 1 1 56C29FCF
 P 8650 5550
@@
 $EndComp
 $Comp
-L GND #PWR074
+L power:GND #PWR074
 U 1 1 56C2A03D
 P 9000 5550
@@
 $EndComp
 $Comp
-L GND #PWR075
+L power:GND #PWR075
 U 1 1 56C2A0AB
 P 9350 5550
@@
 	8650 5550 8650 5450
 $Comp
-L PWR_FLAG #FLG076
+L power:PWR_FLAG #FLG076
 U 1 1 56C2AAAF
 P 9350 4900
@@
 VDD_CC2592
 $Comp
-L VCC #PWR077
+L power:VCC #PWR077
 U 1 1 56C2C769
 P 3800 3750
@@
 LNA_EN
 $Comp
-L Crystal_GND3 X2
+L RCCAR_IF_Board_GPS-rescue:Crystal_GND3-RESCUE-RCCAR_IF_Board_GPS X2
 U 1 1 585F4518
 P 4850 5050
