File: Hardware/RCCAR_IF_Board_GPS/MCU.sch (KiCad schematic (older format))
At the start: 16 parts, among them U1 STM32F40X_LQFP100, X1 8M

Commit message: Added gitignore files
Parts:
- C1, C10, C11, C12, C2, C3, C4, C5, C6, C7, C8, C9: symbol C -> RCCAR_IF_Board_GPS-rescue:C-RESCUE-RCCAR_IF_Board_GPS
- L1: symbol INDUCTOR -> crf_1:INDUCTOR
- R3: symbol R -> RCCAR_IF_Board_GPS-rescue:R-RESCUE-RCCAR_IF_Board_GPS
- U1: symbol STM32F40X_LQFP100 -> crf_1:STM32F40X_LQFP100
- X1: symbol Crystal_GND3 -> RCCAR_IF_Board_GPS-rescue:Crystal_GND3-RESCUE-RCCAR_IF_Board_GPS
Changed lines of the file:
@@
-EESchema Schematic File Version 2
-LIBS:RCCAR_IF_Board_GPS-rescue
-LIBS:power
-LIBS:device
-LIBS:transistors
-LIBS:conn
-LIBS:linear
-LIBS:regul
-LIBS:74xx
-LIBS:cmos4000
-LIBS:adc-dac
-LIBS:memory
-LIBS:xilinx
-LIBS:microcontrollers
-LIBS:dsp
-LIBS:microchip
-LIBS:analog_switches
-LIBS:motorola
-LIBS:texas
-LIBS:intel
-LIBS:audio
-LIBS:interface
-LIBS:digital-audio
-LIBS:philips
-LIBS:display
-LIBS:cypress
-LIBS:siliconi
-LIBS:opto
-LIBS:atmel
-LIBS:contrib
-LIBS:valves
-LIBS:crf_1
-LIBS:dips-s
+EESchema Schematic File Version 4
 LIBS:RCCAR_IF_Board_GPS-cache
 EELAYER 26 0
@@
 $EndDescr
 $Comp
-L VCC #PWR039
+L power:VCC #PWR039
 U 1 1 56AF157C
 P 5100 6100
@@
 $EndComp
 $Comp
-L INDUCTOR L1
+L crf_1:INDUCTOR L1
 U 1 1 56AF1581
 P 6500 6000
@@
 $EndComp
 $Comp
-L VCC #PWR040
+L power:VCC #PWR040
 U 1 1 56AF1582
 P 6500 5600
@@
 $EndComp
 $Comp
-L VCC #PWR041
+L power:VCC #PWR041
 U 1 1 56AF1584
 P 4900 4800
@@
 $EndComp
 $Comp
-L VCC #PWR042
+L power:VCC #PWR042
 U 1 1 56AF1590
 P 6550 1150
@@
 $EndComp
 $Comp
-L PWR_FLAG #FLG043
+L power:PWR_FLAG #FLG043
 U 1 1 56AF1591
 P 6850 6200
@@
 NoConn ~ 4700 2800
 $Comp
-L STM32F40X_LQFP100 U1
+L crf_1:STM32F40X_LQFP100 U1
 U 1 1 56AF1594
 P 3550 3850
@@
 PB15_MOSI2
 $Comp
-L R R3
+L RCCAR_IF_Board_GPS-rescue:R-RESCUE-RCCAR_IF_Board_GPS R3
 U 1 1 56AF1886
 P 6150 5450
@@
 $EndComp
 $Comp
-L C C7
+L RCCAR_IF_Board_GPS-rescue:C-RESCUE-RCCAR_IF_Board_GPS C7
 U 1 1 56AF1A6D
 P 5850 6100
@@
 $EndComp
 $Comp
-L C C6
+L RCCAR_IF_Board_GPS-rescue:C-RESCUE-RCCAR_IF_Board_GPS C6
 U 1 1 56AF268A
 P 5850 5700
@@
 $EndComp
 $Comp
-L GND #PWR044
+L power:GND #PWR044
 U 1 1 56AF2751
 P 6100 6000
@@
 $EndComp
 $Comp
-L C C5
+L RCCAR_IF_Board_GPS-rescue:C-RESCUE-RCCAR_IF_Board_GPS C5
 U 1 1 56AF2977
 P 5800 4750
@@
 $EndComp
 $Comp
-L GND #PWR045
+L power:GND #PWR045
 U 1 1 56AF2A21
 P 6050 4900
@@
 $EndComp
 $Comp
-L GND #PWR046
+L power:GND #PWR046
 U 1 1 56AF2B96
 P 4900 6000
@@
 $EndComp
 $Comp
-L GND #PWR047
+L power:GND #PWR047
 U 1 1 56AF2F6E
 P 5500 6850
@@
 $EndComp
 $Comp
-L C C2
+L RCCAR_IF_Board_GPS-rescue:C-RESCUE-RCCAR_IF_Board_GPS C2
 U 1 1 56AF2FAC
 P 5150 6800
@@
 $EndComp
 $Comp
-L C C3
+L RCCAR_IF_Board_GPS-rescue:C-RESCUE-RCCAR_IF_Board_GPS C3
 U 1 1 56AF3020
 P 5150 7050
@@
 $EndComp
 $Comp
-L C C12
+L RCCAR_IF_Board_GPS-rescue:C-RESCUE-RCCAR_IF_Board_GPS C12
 U 1 1 56AF348F
 P 6800 2300
@@
 $EndComp
 $Comp
-L GND #PWR048
+L power:GND #PWR048
 U 1 1 56AF364A
 P 7050 2500
@@
 $EndComp
 $Comp
-L C C11
+L RCCAR_IF_Board_GPS-rescue:C-RESCUE-RCCAR_IF_Board_GPS C11
 U 1 1 56AF37BB
 P 6800 2050
@@
 $EndComp
 $Comp
-L C C10
+L RCCAR_IF_Board_GPS-rescue:C-RESCUE-RCCAR_IF_Board_GPS C10
 U 1 1 56AF37FC
 P 6800 1800
@@
 $EndComp
 $Comp
-L C C9
+L RCCAR_IF_Board_GPS-rescue:C-RESCUE-RCCAR_IF_Board_GPS C9
 U 1 1 56AF3844
 P 6800 1550
@@
 $EndComp
 $Comp
-L C C8
+L RCCAR_IF_Board_GPS-rescue:C-RESCUE-RCCAR_IF_Board_GPS C8
 U 1 1 56AF3887
 P 6800 1300
@@
 $EndComp
 $Comp
-L C C1
+L RCCAR_IF_Board_GPS-rescue:C-RESCUE-RCCAR_IF_Board_GPS C1
 U 1 1 56AF3AEC
 P 5050 2900
@@
 $EndComp
 $Comp
-L C C4
+L RCCAR_IF_Board_GPS-rescue:C-RESCUE-RCCAR_IF_Board_GPS C4
 U 1 1 56AF3B8E
 P 5750 2900
@@
 $EndComp
 $Comp
-L GND #PWR049
+L power:GND #PWR049
 U 1 1 56AF3C90
 P 6000 2750
@@
 $EndComp
 $Comp
-L GND #PWR050
+L power:GND #PWR050
 U 1 1 56AF4296
 P 4850 3500
@@
 PE1
 $Comp
-L GND #PWR051
+L power:GND #PWR051
 U 1 1 56C88A89
 P 5400 3400
@@
 PB11_SDA2
 $Comp
-L Crystal_GND3 X1
+L RCCAR_IF_Board_GPS-rescue:Crystal_GND3-RESCUE-RCCAR_IF_Board_GPS X1
 U 1 1 585B19B6
 P 5400 3100
