File: Hardware/RCCAR_IF_Board_GPS/MPU9150.sch (KiCad schematic (older format))
At the start: 6 parts, among them U8 MPU9150

Commit message: Added gitignore files
Parts:
- C64, C65, C66, C67, C68: symbol C -> RCCAR_IF_Board_GPS-rescue:C-RESCUE-RCCAR_IF_Board_GPS
- U8: symbol MPU9150 -> crf_1:MPU9150
Changed lines of the file:
@@
-EESchema Schematic File Version 2
-LIBS:RCCAR_IF_Board_GPS-rescue
-LIBS:power
-LIBS:device
-LIBS:transistors
-LIBS:conn
-LIBS:linear
-LIBS:regul
-LIBS:74xx
-LIBS:cmos4000
-LIBS:adc-dac
-LIBS:memory
-LIBS:xilinx
-LIBS:microcontrollers
-LIBS:dsp
-LIBS:microchip
-LIBS:analog_switches
-LIBS:motorola
-LIBS:texas
-LIBS:intel
-LIBS:audio
-LIBS:interface
-LIBS:digital-audio
-LIBS:philips
-LIBS:display
-LIBS:cypress
-LIBS:siliconi
-LIBS:opto
-LIBS:atmel
-LIBS:contrib
-LIBS:valves
-LIBS:crf_1
-LIBS:dips-s
+EESchema Schematic File Version 4
 LIBS:RCCAR_IF_Board_GPS-cache
 EELAYER 26 0
@@
 $EndDescr
 $Comp
-L MPU9150 U8
+L crf_1:MPU9150 U8
 U 1 1 56BD19AD
 P 5400 3800
@@
 Connection ~ 6100 3100
 $Comp
-L VCC #PWR0102
+L power:VCC #PWR0102
 U 1 1 56BD19B1
 P 6500 3050
@@
 	4700 3700 4700 3850
 $Comp
-L C C65
+L RCCAR_IF_Board_GPS-rescue:C-RESCUE-RCCAR_IF_Board_GPS C65
 U 1 1 56BD1B5E
 P 4450 3300
@@
 $EndComp
 $Comp
-L C C64
+L RCCAR_IF_Board_GPS-rescue:C-RESCUE-RCCAR_IF_Board_GPS C64
 U 1 1 56BD1BED
 P 4450 3050
@@
 $EndComp
 $Comp
-L GND #PWR0103
+L power:GND #PWR0103
 U 1 1 56BD1D47
 P 4150 3400
@@
 $EndComp
 $Comp
-L GND #PWR0104
+L power:GND #PWR0104
 U 1 1 56BD1E02
 P 4700 3850
@@
 $EndComp
 $Comp
-L C C66
+L RCCAR_IF_Board_GPS-rescue:C-RESCUE-RCCAR_IF_Board_GPS C66
 U 1 1 56BD1F63
 P 6100 3750
@@
 $EndComp
 $Comp
-L C C67
+L RCCAR_IF_Board_GPS-rescue:C-RESCUE-RCCAR_IF_Board_GPS C67
 U 1 1 56BD1FF4
 P 6300 3750
@@
 $EndComp
 $Comp
-L C C68
+L RCCAR_IF_Board_GPS-rescue:C-RESCUE-RCCAR_IF_Board_GPS C68
 U 1 1 56BD2017
 P 6500 3750
@@
 $EndComp
 $Comp
-L GND #PWR0105
+L power:GND #PWR0105
 U 1 1 56BE1D9B
 P 6500 4600
