File: Hardware/RCCAR_IF_Board_GPS/MPU9250.sch (KiCad schematic (older format))
At the start: 4 parts, among them U14 MPU9250

Commit message: Added gitignore files
Parts:
- C76, C77, C78: symbol C -> RCCAR_IF_Board_GPS-rescue:C-RESCUE-RCCAR_IF_Board_GPS
- U14: symbol MPU9250 -> crf_1:MPU9250
Changed lines of the file:
@@
-EESchema Schematic File Version 2
-LIBS:RCCAR_IF_Board_GPS-rescue
-LIBS:power
-LIBS:device
-LIBS:transistors
-LIBS:conn
-LIBS:linear
-LIBS:regul
-LIBS:74xx
-LIBS:cmos4000
-LIBS:adc-dac
-LIBS:memory
-LIBS:xilinx
-LIBS:microcontrollers
-LIBS:dsp
-LIBS:microchip
-LIBS:analog_switches
-LIBS:motorola
-LIBS:texas
-LIBS:intel
-LIBS:audio
-LIBS:interface
-LIBS:digital-audio
-LIBS:philips
-LIBS:display
-LIBS:cypress
-LIBS:siliconi
-LIBS:opto
-LIBS:atmel
-LIBS:contrib
-LIBS:valves
-LIBS:crf_1
-LIBS:dips-s
+EESchema Schematic File Version 4
 LIBS:RCCAR_IF_Board_GPS-cache
 EELAYER 26 0
@@
 $EndDescr
 $Comp
-L MPU9250 U14
+L crf_1:MPU9250 U14
 U 1 1 59E9DC35
 P 5650 3700
@@
 SDA
 $Comp
-L GND #PWR022
+L power:GND #PWR022
 U 1 1 59E9DD30
 P 4750 4350
@@
 $EndComp
 $Comp
-L VCC #PWR023
+L power:VCC #PWR023
 U 1 1 59E9DDA5
 P 4600 4000
@@
 NoConn ~ 5100 3000
 $Comp
-L C C76
+L RCCAR_IF_Board_GPS-rescue:C-RESCUE-RCCAR_IF_Board_GPS C76
 U 1 1 59E9DE24
 P 6350 4000
@@
 Connection ~ 6350 4300
 $Comp
-L GND #PWR027
+L power:GND #PWR027
 U 1 1 59E9DE84
 P 6350 4500
@@
 Connection ~ 6350 4400
 $Comp
-L C C78
+L RCCAR_IF_Board_GPS-rescue:C-RESCUE-RCCAR_IF_Board_GPS C78
 U 1 1 59E9DEA5
 P 6750 4000
@@
 	6750 4400 6750 4150
 $Comp
-L C C77
+L RCCAR_IF_Board_GPS-rescue:C-RESCUE-RCCAR_IF_Board_GPS C77
 U 1 1 59E9DF54
 P 6550 4000
@@
 Connection ~ 6550 4400
 $Comp
-L VCC #PWR033
+L power:VCC #PWR033
 U 1 1 59E9E01F
 P 6750 2900
