File: Hardware/RCCAR_IF_Board_GPS/RCCAR_IF_Board_GPS.sch (KiCad schematic (older format))
At the start: 35 parts, among them P1 POWER, P13 USB_UBLOX, P2 USB_STM, P3 I2C, P4 UART, P5 NRF_SPI, P6 SWD, P7 ADC_GPIO, P8 CAN, P9 CAN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

Commit message: Updated PCB with MPU9250
Parts:
- P13, P2: symbol USB_OTG -> USB_OTG-RESCUE-RCCAR_IF_Board_GPS
Connections:
- wire segments 191 -> 195
Other:
- moved on the sheet: C61, C62, D1, D2, D3, D4, P1, P3, P4, P5, P6, P7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

Commit message: Added gitignore files
Parts:
- C61, C62: symbol C -> RCCAR_IF_Board_GPS-rescue:C-RESCUE-RCCAR_IF_Board_GPS
- D1, D2, D3, D4: symbol LED -> RCCAR_IF_Board_GPS-rescue:LED-RESCUE-RCCAR_IF_Board_GPS
- P1, P3, P4, P8, P9: symbol CONN_01X04 -> RCCAR_IF_Board_GPS-rescue:CONN_01X04-RESCUE-RCCAR_IF_Board_GPS
- P13, P2: symbol USB_OTG-RESCUE-RCCAR_IF_Board_GPS -> RCCAR_IF_Board_GPS-rescue:USB_OTG-RESCUE-RCCAR_IF_Board_GPS
- P5: symbol CONN_01X08 -> RCCAR_IF_Board_GPS-rescue:CONN_01X08-RESCUE-RCCAR_IF_Board_GPS
- P6, P7: symbol CONN_01X06 -> RCCAR_IF_Board_GPS-rescue:CONN_01X06-RESCUE-RCCAR_IF_Board_GPS
- R1, R10, R2, R21, R22, R23, R24, R25, R26, R27, R35, R6, R7, R9: symbol R -> RCCAR_IF_Board_GPS-rescue:R-RESCUE-RCCAR_IF_Board_GPS
- SW1: symbol DIPS_08 -> dips-s:DIPS_08
- U10, U11, U9: symbol SWITCH_SPDT -> crf_1:SWITCH_SPDT
- U12: symbol AP131-33 -> RCCAR_IF_Board_GPS-rescue:AP131-33-RESCUE-RCCAR_IF_Board_GPS
