File: Hardware/RCCAR_IF_Board_GPS/SERVO_IO.sch (KiCad schematic (older format))
At the start: 10 parts, among them P11 OUT_1, P12 OUT_2, P14 OUT_3, P15 OUT_4

Commit message: Added gitignore files
Parts:
- P11, P12, P14, P15: symbol CONN_01X03 -> RCCAR_IF_Board_GPS-rescue:CONN_01X03-RESCUE-RCCAR_IF_Board_GPS
- R15, R16, R17, R18, R33, R34: symbol R -> RCCAR_IF_Board_GPS-rescue:R-RESCUE-RCCAR_IF_Board_GPS
Changed lines of the file:
@@
-EESchema Schematic File Version 2
-LIBS:RCCAR_IF_Board_GPS-rescue
-LIBS:power
-LIBS:device
-LIBS:transistors
-LIBS:conn
-LIBS:linear
-LIBS:regul
-LIBS:74xx
-LIBS:cmos4000
-LIBS:adc-dac
-LIBS:memory
-LIBS:xilinx
-LIBS:microcontrollers
-LIBS:dsp
-LIBS:microchip
-LIBS:analog_switches
-LIBS:motorola
-LIBS:texas
-LIBS:intel
-LIBS:audio
-LIBS:interface
-LIBS:digital-audio
-LIBS:philips
-LIBS:display
-LIBS:cypress
-LIBS:siliconi
-LIBS:opto
-LIBS:atmel
-LIBS:contrib
-LIBS:valves
-LIBS:crf_1
-LIBS:dips-s
+EESchema Schematic File Version 4
 LIBS:RCCAR_IF_Board_GPS-cache
 EELAYER 26 0
@@
 $EndDescr
 $Comp
-L CONN_01X03 P11
+L RCCAR_IF_Board_GPS-rescue:CONN_01X03-RESCUE-RCCAR_IF_Board_GPS P11
 U 1 1 56C05596
 P 6350 3250
@@
 $EndComp
 $Comp
-L CONN_01X03 P12
+L RCCAR_IF_Board_GPS-rescue:CONN_01X03-RESCUE-RCCAR_IF_Board_GPS P12
 U 1 1 56C0560F
 P 6350 3700
@@
 Connection ~ 5150 3350
 $Comp
-L R R16
+L RCCAR_IF_Board_GPS-rescue:R-RESCUE-RCCAR_IF_Board_GPS R16
 U 1 1 56C057DB
 P 5150 2800
@@
 $EndComp
 $Comp
-L R R15
+L RCCAR_IF_Board_GPS-rescue:R-RESCUE-RCCAR_IF_Board_GPS R15
 U 1 1 56C0582C
 P 4950 2800
@@
 	4950 2950 4950 3350
 $Comp
-L GND #PWR097
+L power:GND #PWR097
 U 1 1 56C058BF
 P 4750 2750
@@
 Bridge options\nfor internal supply
 $Comp
-L +5V #PWR098
+L power:+5V #PWR098
 U 1 1 56C0673F
 P 5150 2450
@@
 $EndComp
 $Comp
-L R R33
+L RCCAR_IF_Board_GPS-rescue:R-RESCUE-RCCAR_IF_Board_GPS R33
 U 1 1 56C1A2B5
 P 5950 3150
@@
 	6100 3150 6150 3150
 $Comp
-L R R34
+L RCCAR_IF_Board_GPS-rescue:R-RESCUE-RCCAR_IF_Board_GPS R34
 U 1 1 56C1A788
 P 5950 3600
@@
 	5750 3600 5800 3600
 $Comp
-L CONN_01X03 P14
+L RCCAR_IF_Board_GPS-rescue:CONN_01X03-RESCUE-RCCAR_IF_Board_GPS P14
 U 1 1 585DB678
 P 6350 4150
@@
 OUT_3
 $Comp
-L R R17
+L RCCAR_IF_Board_GPS-rescue:R-RESCUE-RCCAR_IF_Board_GPS R17
 U 1 1 585DB681
 P 5950 4050
@@
 	5750 4050 5800 4050
 $Comp
-L CONN_01X03 P15
+L RCCAR_IF_Board_GPS-rescue:CONN_01X03-RESCUE-RCCAR_IF_Board_GPS P15
 U 1 1 585DB92D
 P 6350 4600
@@
 OUT_4
 $Comp
-L R R18
+L RCCAR_IF_Board_GPS-rescue:R-RESCUE-RCCAR_IF_Board_GPS R18
 U 1 1 585DB934
 P 5950 4500
