File: Hardware/RCCAR_IF_Board_GPS/VREG.sch (KiCad schematic (older format))
At the start: 20 parts, among them U5 MCP16311/2, U6 MCP16311/2

Commit message: Added gitignore files
Parts:
- C52, C53, C54, C55, C57, C58, C59, C60: symbol C -> RCCAR_IF_Board_GPS-rescue:C-RESCUE-RCCAR_IF_Board_GPS
- C56, C69: symbol CP1 -> RCCAR_IF_Board_GPS-rescue:CP1-RESCUE-RCCAR_IF_Board_GPS
- L14, L16: symbol INDUCTOR -> crf_1:INDUCTOR
- R13, R14, R28, R29, R30, R31: symbol R -> RCCAR_IF_Board_GPS-rescue:R-RESCUE-RCCAR_IF_Board_GPS
- U5, U6: symbol MCP16311/2 -> RCCAR_IF_Board_GPS-rescue:MCP16311_2-RESCUE-RCCAR_IF_Board_GPS
Changed lines of the file:
@@
-EESchema Schematic File Version 2
-LIBS:RCCAR_IF_Board_GPS-rescue
-LIBS:power
-LIBS:device
-LIBS:transistors
-LIBS:conn
-LIBS:linear
-LIBS:regul
-LIBS:74xx
-LIBS:cmos4000
-LIBS:adc-dac
-LIBS:memory
-LIBS:xilinx
-LIBS:microcontrollers
-LIBS:dsp
-LIBS:microchip
-LIBS:analog_switches
-LIBS:motorola
-LIBS:texas
-LIBS:intel
-LIBS:audio
-LIBS:interface
-LIBS:digital-audio
-LIBS:philips
-LIBS:display
-LIBS:cypress
-LIBS:siliconi
-LIBS:opto
-LIBS:atmel
-LIBS:contrib
-LIBS:valves
-LIBS:crf_1
-LIBS:dips-s
+EESchema Schematic File Version 4
 LIBS:RCCAR_IF_Board_GPS-cache
 EELAYER 26 0
@@
 $EndDescr
 $Comp
-L MCP16311/2 U5
+L RCCAR_IF_Board_GPS-rescue:MCP16311_2-RESCUE-RCCAR_IF_Board_GPS U5
 U 1 1 56BFBAD5
 P 5400 2650
@@
 $EndComp
 $Comp
-L INDUCTOR L14
+L crf_1:INDUCTOR L14
 U 1 1 56BFBAD8
 P 6800 2700
@@
 3.3V
 $Comp
-L C C52
+L RCCAR_IF_Board_GPS-rescue:C-RESCUE-RCCAR_IF_Board_GPS C52
 U 1 1 56BFC39E
 P 4400 3050
@@
 $EndComp
 $Comp
-L C C53
+L RCCAR_IF_Board_GPS-rescue:C-RESCUE-RCCAR_IF_Board_GPS C53
 U 1 1 56BFC4C1
 P 4650 3050
@@
 $EndComp
 $Comp
-L C C55
+L RCCAR_IF_Board_GPS-rescue:C-RESCUE-RCCAR_IF_Board_GPS C55
 U 1 1 56BFC55D
 P 6900 3050
@@
 $EndComp
 $Comp
-L CP1 C56
+L RCCAR_IF_Board_GPS-rescue:CP1-RESCUE-RCCAR_IF_Board_GPS C56
 U 1 1 56BFC607
 P 7150 3050
@@
 $EndComp
 $Comp
-L GND #PWR095
+L power:GND #PWR095
 U 1 1 56BFC6AC
 P 6100 3400
@@
 $EndComp
 $Comp
-L C C54
+L RCCAR_IF_Board_GPS-rescue:C-RESCUE-RCCAR_IF_Board_GPS C54
 U 1 1 56BFC7B9
 P 6400 2450
@@
 $EndComp
 $Comp
-L R R14
+L RCCAR_IF_Board_GPS-rescue:R-RESCUE-RCCAR_IF_Board_GPS R14
 U 1 1 56BFC87E
 P 5700 2150
@@
 $EndComp
 $Comp
-L R R13
+L RCCAR_IF_Board_GPS-rescue:R-RESCUE-RCCAR_IF_Board_GPS R13
 U 1 1 56BFC8C4
 P 5000 2150
@@
 $EndComp
 $Comp
-L MCP16311/2 U6
+L RCCAR_IF_Board_GPS-rescue:MCP16311_2-RESCUE-RCCAR_IF_Board_GPS U6
 U 1 1 56BF90CD
 P 5400 4600
@@
 $EndComp
 $Comp
-L INDUCTOR L16
+L crf_1:INDUCTOR L16
 U 1 1 56BF90D3
 P 6800 4650
@@
 Connection ~ 4550 4750
 $Comp
-L C C57
+L RCCAR_IF_Board_GPS-rescue:C-RESCUE-RCCAR_IF_Board_GPS C57
 U 1 1 56BF910A
 P 4400 5000
@@
 $EndComp
 $Comp
-L C C58
+L RCCAR_IF_Board_GPS-rescue:C-RESCUE-RCCAR_IF_Board_GPS C58
 U 1 1 56BF9110
 P 4650 5000
@@
 $EndComp
 $Comp
-L C C60
+L RCCAR_IF_Board_GPS-rescue:C-RESCUE-RCCAR_IF_Board_GPS C60
 U 1 1 56BF9116
 P 6900 5000
@@
 $EndComp
 $Comp
-L CP1 C69
+L RCCAR_IF_Board_GPS-rescue:CP1-RESCUE-RCCAR_IF_Board_GPS C69
 U 1 1 56BF911C
 P 7150 5000
@@
 $EndComp
 $Comp
-L GND #PWR096
+L power:GND #PWR096
 U 1 1 56BF9122
 P 6100 5350
@@
 $EndComp
 $Comp
-L C C59
+L RCCAR_IF_Board_GPS-rescue:C-RESCUE-RCCAR_IF_Board_GPS C59
 U 1 1 56BF9128
 P 6400 4400
@@
 $EndComp
 $Comp
-L R R31
+L RCCAR_IF_Board_GPS-rescue:R-RESCUE-RCCAR_IF_Board_GPS R31
 U 1 1 56BF912E
 P 5700 4100
@@
 $EndComp
 $Comp
-L R R30
+L RCCAR_IF_Board_GPS-rescue:R-RESCUE-RCCAR_IF_Board_GPS R30
 U 1 1 56BF9134
 P 5000 4100
@@
 5V
 $Comp
-L R R28
+L RCCAR_IF_Board_GPS-rescue:R-RESCUE-RCCAR_IF_Board_GPS R28
 U 1 1 56BF97D6
 P 3950 4350
@@
 $EndComp
 $Comp
-L R R29
+L RCCAR_IF_Board_GPS-rescue:R-RESCUE-RCCAR_IF_Board_GPS R29
 U 1 1 56BF9895
 P 3950 4550
