File: Hardware/RCCAR_IF_Board_GPS/ublox.sch (KiCad schematic (older format))
At the start: 6 parts, among them J3 SMA, U13 ublox_neo_m8p

Commit message: Updated PCB with MPU9250
Parts:
- R20: value 10R -> 4.7R
Changed lines of the file:
@@
 EESchema Schematic File Version 2
+LIBS:RCCAR_IF_Board_GPS-rescue
 LIBS:power
 LIBS:device
@@
 $Descr A4 11693 8268
 encoding utf-8
-Sheet 9 9
+Sheet 9 10
 Title "M8T/M8P"
 Date ""
 Rev "A"
-Comp "SP"
+Comp "RISE"
 Comment1 ""
 Comment2 ""
@@
 P 7200 3400
 F 0 "R20" V 7300 3400 50  0000 C CNN
-F 1 "10R" V 7100 3400 50  0000 C CNN
+F 1 "4.7R" V 7100 3400 50  0000 C CNN
 F 2 "Resistors_SMD:R_0603" V 7130 3400 50  0001 C CNN
 F 3 "" H 7200 3400 50  0000 C CNN

Commit message: Added gitignore files
Parts:
- C74, C75: symbol C -> RCCAR_IF_Board_GPS-rescue:C-RESCUE-RCCAR_IF_Board_GPS
- J3: symbol SMA -> crf_1:SMA
- L18: symbol L -> RCCAR_IF_Board_GPS-rescue:L-RESCUE-RCCAR_IF_Board_GPS
- R20: symbol R -> RCCAR_IF_Board_GPS-rescue:R-RESCUE-RCCAR_IF_Board_GPS
- U13: symbol ublox_neo_m8p -> crf_1:ublox_neo_m8p
Changed lines of the file:
@@
-EESchema Schematic File Version 2
-LIBS:RCCAR_IF_Board_GPS-rescue
-LIBS:power
-LIBS:device
-LIBS:transistors
-LIBS:conn
-LIBS:linear
-LIBS:regul
-LIBS:74xx
-LIBS:cmos4000
-LIBS:adc-dac
-LIBS:memory
-LIBS:xilinx
-LIBS:microcontrollers
-LIBS:dsp
-LIBS:microchip
-LIBS:analog_switches
-LIBS:motorola
-LIBS:texas
-LIBS:intel
-LIBS:audio
-LIBS:interface
-LIBS:digital-audio
-LIBS:philips
-LIBS:display
-LIBS:cypress
-LIBS:siliconi
-LIBS:opto
-LIBS:atmel
-LIBS:contrib
-LIBS:valves
-LIBS:crf_1
-LIBS:dips-s
+EESchema Schematic File Version 4
 LIBS:RCCAR_IF_Board_GPS-cache
 EELAYER 26 0
@@
 $EndDescr
 $Comp
-L ublox_neo_m8p U13
+L crf_1:ublox_neo_m8p U13
 U 1 1 585F12E3
 P 5650 3700
@@
 $EndComp
 $Comp
-L C C74
+L RCCAR_IF_Board_GPS-rescue:C-RESCUE-RCCAR_IF_Board_GPS C74
 U 1 1 585F135A
 P 4450 4450
@@
 	4450 4600 4450 4850
 $Comp
-L GND #PWR0106
+L power:GND #PWR0106
 U 1 1 585F1434
 P 4450 4850
@@
 Connection ~ 4450 4750
 $Comp
-L VCC #PWR0107
+L power:VCC #PWR0107
 U 1 1 585F1463
 P 4450 4050
@@
 RTK_STAT
 $Comp
-L SMA J3
+L crf_1:SMA J3
 U 1 1 585F2744
 P 6800 2700
@@
 	6700 3200 6700 2800
 $Comp
-L L L18
+L RCCAR_IF_Board_GPS-rescue:L-RESCUE-RCCAR_IF_Board_GPS L18
 U 1 1 585F28EA
 P 7350 3200
@@
 $EndComp
 $Comp
-L C C75
+L RCCAR_IF_Board_GPS-rescue:C-RESCUE-RCCAR_IF_Board_GPS C75
 U 1 1 585F35FF
 P 7600 3600
@@
 $EndComp
 $Comp
-L R R20
+L RCCAR_IF_Board_GPS-rescue:R-RESCUE-RCCAR_IF_Board_GPS R20
 U 1 1 585F3849
 P 7200 3400
@@
 Connection ~ 7600 3400
 $Comp
-L GND #PWR0108
+L power:GND #PWR0108
 U 1 1 585F39D8
 P 7600 3900
@@
 Connection ~ 7000 2700
 $Comp
-L GND #PWR0109
+L power:GND #PWR0109
 U 1 1 585F6B31
 P 7000 2800
@@
 Connection ~ 6950 3300
 $Comp
-L GND #PWR0110
+L power:GND #PWR0110
 U 1 1 585F6C2B
 P 6950 3500
@@
 $EndComp
 $Comp
-L GND #PWR0111
+L power:GND #PWR0111
 U 1 1 585F6CC6
 P 4300 3450
